Commit message: MG: working

File: follower_description/urdf/gazebo.urdf.xacro (robot description, xacro)
@@ -12,10 +12,10 @@
                 <wheelSeparation>0.4</wheelSeparation>
                 <wheelDiameter>0.215</wheelDiameter>
-                <robotBaseFrame>base_link</robotBaseFrame>
+                <robotBaseFrame>${prefix}/base_link</robotBaseFrame>
                 <MaxForce>5.0</MaxForce>
                 <torque>200</torque>
                 <commandTopic>cmd_vel</commandTopic>
                 <odometryTopic>odom</odometryTopic>
-                <odometryFrame>odom</odometryFrame>
+                <odometryFrame>${prefix}/odom</odometryFrame>
                 <broadcastTF>1</broadcastTF>
             </plugin>
@@ -41,3 +41,135 @@
         </gazebo>
     </xacro:macro>
+  <xacro:macro name="gazebo_d435" params="camera_name reference_link topics_ns depth_optical_frame color_optical_frame infrared1_optical_frame infrared2_optical_frame publish_pointcloud:=true" >
+    <!-- Load parameters to model's main link-->
+    <xacro:property name="deg_to_rad" value="0.01745329251994329577" />
+    <gazebo reference="${reference_link}">
+      <self_collide>0</self_collide>
+      <enable_wind>0</enable_wind>
+      <kinematic>0</kinematic>
+      <gravity>1</gravity>
+      <!--<mu>1</mu>-->
+      <mu2>1</mu2>
+      <fdir1>0 0 0</fdir1>
+      <!--<slip1>0</slip1>
+      <slip2>0</slip2>-->
+      <kp>1e+13</kp>
+      <kd>1</kd>
+      <!--<max_vel>0.01</max_vel>
+      <min_depth>0</min_depth>-->
+      <sensor name="${camera_name}color" type="camera">
+        <camera name="${camera_name}">
+          <horizontal_fov>${69.4*deg_to_rad}</horizontal_fov>
+          <image>
+            <width>640</width>
+            <height>480</height>
+            <format>RGB_INT8</format>
+          </image>
+          <clip>
+            <near>0.1</near>
+            <far>100</far>
+          </clip>
+          <noise>
+            <type>gaussian</type>
+            <mean>0.0</mean>
+            <stddev>0.007</stddev>
+          </noise>
+        </camera>
+        <always_on>1</always_on>
+        <update_rate>30</update_rate>
+        <visualize>1</visualize>
+      </sensor>
+      <sensor name="${camera_name}ired1" type="camera">
+        <camera name="${camera_name}">
+          <horizontal_fov>${85.2*deg_to_rad}</horizontal_fov>
+          <image>
+            <width>1280</width>
+            <height>720</height>
+            <format>L_INT8</format>
+          </image>
+          <clip>
+            <near>0.1</near>
+            <far>100</far>
+          </clip>
+          <noise>
+            <type>gaussian</type>
+            <mean>0.0</mean>
+            <stddev>0.05</stddev>
+          </noise>
+        </camera>
+        <always_on>1</always_on>
+        <update_rate>90</update_rate>
+        <visualize>0</visualize>
+      </sensor>
+      <sensor name="${camera_name}ired2" type="camera">
+        <camera name="${camera_name}">
+          <horizontal_fov>${85.2*deg_to_rad}</horizontal_fov>
+          <image>
+            <width>1280</width>
+            <height>720</height>
+            <format>L_INT8</format>
+          </image>
+          <clip>
+            <near>0.1</near>
+            <far>100</far>
+          </clip>
+          <noise>
+            <type>gaussian</type>
+            <mean>0.0</mean>
+            <stddev>0.05</stddev>
+          </noise>
+        </camera>
+        <always_on>1</always_on>
+        <update_rate>90</update_rate>
+        <visualize>0</visualize>
+      </sensor>
+      <sensor name="${camera_name}depth" type="depth">
+        <camera name="${camera_name}">
+          <horizontal_fov>${85.2*deg_to_rad}</horizontal_fov>
+          <image>
+            <width>1280</width>
+            <height>720</height>
+          </image>
+          <clip>
+            <near>0.1</near>
+            <far>100</far>
+          </clip>
+          <noise>
+            <type>gaussian</type>
+            <mean>0.0</mean>
+            <stddev>0.100</stddev>
+          </noise>
+        </camera>
+        <always_on>1</always_on>
+        <update_rate>90</update_rate>
+        <visualize>0</visualize>
+      </sensor>
+    </gazebo>
+    <gazebo>
+      <plugin name="${topics_ns}" filename="librealsense_gazebo_plugin.so">
+        <prefix>${camera_name}</prefix>
+        <depthUpdateRate>30.0</depthUpdateRate>
+        <colorUpdateRate>30.0</colorUpdateRate>
+        <infraredUpdateRate>30.0</infraredUpdateRate>
+        <depthTopicName>depth/image_raw</depthTopicName>
+        <depthCameraInfoTopicName>depth/camera_info</depthCameraInfoTopicName>
+        <colorTopicName>color/image_raw</colorTopicName>
+        <colorCameraInfoTopicName>color/camera_info</colorCameraInfoTopicName>
+        <infrared1TopicName>infra1/image_raw</infrared1TopicName>
+        <infrared1CameraInfoTopicName>infra1/camera_info</infrared1CameraInfoTopicName>
+        <infrared2TopicName>infra2/image_raw</infrared2TopicName>
+        <infrared2CameraInfoTopicName>infra2/camera_info</infrared2CameraInfoTopicName>
+        <colorOpticalframeName>${color_optical_frame}</colorOpticalframeName>
+        <depthOpticalframeName>${depth_optical_frame}</depthOpticalframeName>
+        <infrared1OpticalframeName>${infrared1_optical_frame}</infrared1OpticalframeName>
+        <infrared2OpticalframeName>${infrared2_optical_frame}</infrared2OpticalframeName>
+        <rangeMinDepth>0.2</rangeMinDepth>
+        <rangeMaxDepth>10.0</rangeMaxDepth>
+        <pointCloud>${publish_pointcloud}</pointCloud>
+        <pointCloudTopicName>depth/color/points</pointCloudTopicName>
+        <pointCloudCutoff>0.25</pointCloudCutoff>
+        <pointCloudCutoffMax>9.0</pointCloudCutoffMax>
+      </plugin>
+    </gazebo>
+  </xacro:macro>
 </robot>

File: follower_description/urdf/pioneer3at.urdf.xacro (robot description, xacro)
@@ -6,4 +6,10 @@
 <robot name="pioneer3at" xmlns:xacro="http://ros.org/wiki/xacro">
   <xacro:macro name="pioneer3at" params="prefix">
+  <link name="base_footprint">
+   </link>
+  <joint name="base_footprint_joint" type="fixed">
+     <parent link="base_footprint"/>
+     <child link="base_link"/>
+  </joint>
     <!-- Chassis -->
     <link name="base_link">
@@ -24,5 +30,5 @@
         <origin rpy="0 0 0" xyz="0 0 0.177"/>
         <geometry name="pioneer_geom">
-          <mesh filename="package://follower_description/meshes/p3at_meshes/chassis.stl"/>
+          <mesh filename="package://follower_description/meshes/p3at/chassis.stl"/>
         </geometry>
         <material name="ChassisRed">
@@ -33,5 +39,5 @@
         <origin rpy="0 0 0" xyz="0 0 0.177"/>
         <geometry>
-          <mesh filename="package://follower_description/meshes/p3at_meshes/chassis.stl"/>
+          <mesh filename="package://follower_description/meshes/p3at/chassis.stl"/>
         </geometry>
       </collision>
@@ -50,5 +56,5 @@
         <origin rpy="0 0 0" xyz="0 0 0"/>
         <geometry name="pioneer_geom">
-          <mesh filename="package://follower_description/meshes/p3at_meshes/top.stl"/>
+          <mesh filename="package://follower_description/meshes/p3at/top.stl"/>
         </geometry>
         <material name="TopBlack">
@@ -75,5 +81,5 @@
         <origin rpy="0 0 0" xyz="0 0 0"/>
         <geometry name="pioneer_geom">
-          <mesh filename="package://follower_description/meshes/p3at_meshes/front_sonar.stl"/>
+          <mesh filename="package://follower_description/meshes/p3at/front_sonar.stl"/>
         </geometry>
         <material name="SonarYellow">
@@ -99,5 +105,5 @@
         <origin rpy="0 0 0" xyz="0 0 0"/>
         <geometry name="pioneer_geom">
-          <mesh filename="package://follower_description/meshes/p3at_meshes/back_sonar.stl"/>
+          <mesh filename="package://follower_description/meshes/p3at/back_sonar.stl"/>
         </geometry>
         <material name="SonarYellow">
@@ -124,5 +130,5 @@
         <origin rpy="0 0 0" xyz="0 0 0"/>
         <geometry name="pioneer_geom">
-          <mesh filename="package://follower_description/meshes/p3at_meshes/axle.stl"/>
+          <mesh filename="package://follower_description/meshes/p3at/axle.stl"/>
         </geometry>
         <material name="AxleGrey">
@@ -148,5 +154,5 @@
         <origin rpy="0 0 0" xyz="0 0 0"/>
         <geometry name="pioneer_geom">
-          <mesh filename="package://follower_description/meshes/p3at_meshes/left_hubcap.stl"/>
+          <mesh filename="package://follower_description/meshes/p3at/left_hubcap.stl"/>
         </geometry>
         <material name="HubcapYellow">
@@ -173,5 +179,5 @@
         <origin rpy="0 0 0" xyz="0 0 0"/>
         <geometry name="pioneer_geom">
-          <mesh filename="package://follower_description/meshes/p3at_meshes/wheel.stl"/>
+          <mesh filename="package://follower_description/meshes/p3at/wheel.stl"/>
         </geometry>
         <material name="WheelBlack">
@@ -182,5 +188,5 @@
         <origin rpy="-1.57079635 0 0" xyz="0 0 0"/>
         <geometry>
-          <!--mesh filename="package://follower_description/meshes/p3at_meshes/wheel.stl"/-->
+          <!--mesh filename="package://follower_description/meshes/p3at/wheel.stl"/-->
           <cylinder length="0.075" radius="0.111"/>
         </geometry>
@@ -209,5 +215,5 @@
         <origin rpy="0 0 0" xyz="0 0 0"/>
         <geometry name="pioneer_geom">
-          <mesh filename="package://follower_description/meshes/p3at_meshes/axle.stl"/>
+          <mesh filename="package://follower_description/meshes/p3at/axle.stl"/>
         </geometry>
         <material name="AxleGrey">
@@ -218,5 +224,5 @@
         <origin rpy="0 0 0" xyz="0 0 0"/>
         <geometry>
-          <mesh filename="package://follower_description/meshes/p3at_meshes/axle.stl"/>
+          <mesh filename="package://follower_description/meshes/p3at/axle.stl"/>
         </geometry>
       </collision>
@@ -239,5 +245,5 @@
         <origin rpy="0 0 0" xyz="0 0 0"/>
         <geometry name="pioneer_geom">
-          <mesh filename="package://follower_description/meshes/p3at_meshes/left_hubcap.stl"/>
+          <mesh filename="package://follower_description/meshes/p3at/left_hubcap.stl"/>
         </geometry>
         <material name="HubcapYellow"/>
@@ -246,5 +252,5 @@
         <origin rpy="0 0 0" xyz="0 0 0"/>
         <geometry>
-          <mesh filename="package://follower_description/meshes/p3at_meshes/left_hubcap.stl"/>
+          <mesh filename="package://follower_description/meshes/p3at/left_hubcap.stl"/>
         </geometry>
       </collision>
@@ -267,5 +273,5 @@
         <origin rpy="0 0 0" xyz="0 0 0"/>
         <geometry name="pioneer_geom">
-          <mesh filename="package://follower_description/meshes/p3at_meshes/wheel.stl"/>
+          <mesh filename="package://follower_description/meshes/p3at/wheel.stl"/>
         </geometry>
         <material name="WheelBlack"/>
@@ -274,5 +280,5 @@
         <origin rpy="-1.57079635 0 0" xyz="0 0 0"/>
         <geometry>
-          <!--mesh filename="package://follower_description/meshes/p3at_meshes/wheel.stl"/-->
+          <!--mesh filename="package://follower_description/meshes/p3at/wheel.stl"/-->
           <cylinder length="0.075" radius="0.111"/>
         </geometry>
@@ -301,5 +307,5 @@
         <origin rpy="0 0 0" xyz="0 0 0"/>
         <geometry name="pioneer_geom">
-          <mesh filename="package://follower_description/meshes/p3at_meshes/axle.stl"/>
+          <mesh filename="package://follower_description/meshes/p3at/axle.stl"/>
         </geometry>
         <material name="AxleGrey">
@@ -325,5 +331,5 @@
         <origin rpy="0 0 0" xyz="0 0 0"/>
         <geometry name="pioneer_geom">
-          <mesh filename="package://follower_description/meshes/p3at_meshes/right_hubcap.stl"/>
+          <mesh filename="package://follower_description/meshes/p3at/right_hubcap.stl"/>
         </geometry>
         <material name="HubcapYellow">
@@ -350,5 +356,5 @@
         <origin rpy="0 0 0" xyz="0 0 0"/>
         <geometry name="pioneer_geom">
-          <mesh filename="package://follower_description/meshes/p3at_meshes/wheel.stl"/>
+          <mesh filename="package://follower_description/meshes/p3at/wheel.stl"/>
         </geometry>
         <material name="WheelBlack">
@@ -359,5 +365,5 @@
         <origin rpy="-1.57079635 0 0" xyz="0 0 0"/>
         <geometry>
-          <!--mesh filename="package://follower_description/meshes/p3at_meshes/wheel.stl"/-->
+          <!--mesh filename="package://follower_description/meshes/p3at/wheel.stl"/-->
           <cylinder length="0.075" radius="0.111"/>
         </geometry>
@@ -386,5 +392,5 @@
         <origin rpy="0 0 0" xyz="0 0 0"/>
         <geometry name="pioneer_geom">
-          <mesh filename="package://follower_description/meshes/p3at_meshes/axle.stl"/>
+          <mesh filename="package://follower_description/meshes/p3at/axle.stl"/>
         </geometry>
         <material name="AxleGrey">
@@ -395,5 +401,5 @@
         <origin rpy="0 0 0" xyz="0 0 0"/>
         <geometry>
-          <mesh filename="package://follower_description/meshes/p3at_meshes/axle.stl"/>
+          <mesh filename="package://follower_description/meshes/p3at/axle.stl"/>
         </geometry>
       </collision>
@@ -416,5 +422,5 @@
         <origin rpy="0 0 0" xyz="0 0 0"/>
         <geometry name="pioneer_geom">
-          <mesh filename="package://follower_description/meshes/p3at_meshes/right_hubcap.stl"/>
+          <mesh filename="package://follower_description/meshes/p3at/right_hubcap.stl"/>
         </geometry>
         <material name="HubcapYellow"/>
@@ -423,5 +429,5 @@
         <origin rpy="0 0 0" xyz="0 0 0"/>
         <geometry>
-          <mesh filename="package://follower_description/meshes/p3at_meshes/right_hubcap.stl"/>
+          <mesh filename="package://follower_description/meshes/p3at/right_hubcap.stl"/>
         </geometry>
       </collision>
@@ -444,5 +450,5 @@
         <origin rpy="0 0 0" xyz="0 0 0"/>
         <geometry name="pioneer_geom">
-          <mesh filename="package://follower_description/meshes/p3at_meshes/wheel.stl"/>
+          <mesh filename="package://follower_description/meshes/p3at/wheel.stl"/>
         </geometry>
         <material name="WheelBlack"/>
@@ -451,5 +457,5 @@
         <origin rpy="-1.57079635 0 0" xyz="0 0 0"/>
         <geometry>
-          <!--mesh filename="package://follower_description/meshes/p3at_meshes/wheel.stl"/-->
+          <!--mesh filename="package://follower_description/meshes/p3at/wheel.stl"/-->
           <cylinder length="0.075" radius="0.111"/>
         </geometry>
@@ -468,4 +474,5 @@
       <child link="p3at_back_right_wheel"/>
     </joint>
+  <!-- Gazebo -->
   </xacro:macro>
 </robot>
