Commit message: MG: fixed tf

File: follower_description/urdf/gazebo.urdf.xacro (robot description, xacro)
@@ -6,11 +6,11 @@
                 <updateRate>100.0</updateRate>
                 <robotNamespace>${prefix}</robotNamespace>
-                <leftFrontJoint>p3at_front_left_wheel_joint</leftFrontJoint>
-                <rightFrontJoint>p3at_front_right_wheel_joint</rightFrontJoint>
-                <leftRearJoint>p3at_back_left_wheel_joint</leftRearJoint>
-                <rightRearJoint>p3at_back_right_wheel_joint</rightRearJoint>
+                <leftFrontJoint>${prefix}/p3at_front_left_wheel_joint</leftFrontJoint>
+                <rightFrontJoint>${prefix}/p3at_front_right_wheel_joint</rightFrontJoint>
+                <leftRearJoint>${prefix}/p3at_back_left_wheel_joint</leftRearJoint>
+                <rightRearJoint>${prefix}/p3at_back_right_wheel_joint</rightRearJoint>
                 <wheelSeparation>0.4</wheelSeparation>
                 <wheelDiameter>0.215</wheelDiameter>
-                <robotBaseFrame>${prefix}/base_link</robotBaseFrame>
+                <robotBaseFrame>${prefix}/base_footprint</robotBaseFrame>
                 <MaxForce>5.0</MaxForce>
                 <torque>200</torque>
@@ -21,4 +21,7 @@
             </plugin>
         </gazebo>
+      <!-- <gazebo>
+        <plugin name="joint_state_publisher" filename="libgazebo_ros_joint_state_publisher.so" />
+      </gazebo> -->
     </xacro:macro>
     <xacro:macro name='p3at_wheel' params='link'>

File: follower_description/urdf/pioneer3at.urdf.xacro (robot description, xacro)
@@ -6,12 +6,12 @@
 <robot name="pioneer3at" xmlns:xacro="http://ros.org/wiki/xacro">
   <xacro:macro name="pioneer3at" params="prefix">
-  <link name="base_footprint">
+  <link name="${prefix}/base_footprint">
    </link>
-  <joint name="base_footprint_joint" type="fixed">
-     <parent link="base_footprint"/>
-     <child link="base_link"/>
+  <joint name="${prefix}/base_footprint_joint" type="fixed">
+     <parent link="${prefix}/base_footprint"/>
+     <child link="${prefix}/base_link"/>
   </joint>
     <!-- Chassis -->
-    <link name="base_link">
+    <link name="${prefix}/base_link">
       <!--  For pointers on inertial and gazebo-related parameters see
             * http://wiki.ros.org/urdf/Tutorials/Adding%20Physical%20and%20Collision%20Properties%20to%20a%20URDF%20Model
@@ -43,9 +43,9 @@
       </collision>
     </link>
-    <gazebo reference="base_link">
+    <gazebo reference="${prefix}/base_link">
       <material value="Gazebo/Red"/>
     </gazebo>
     <!-- Top -->
-    <link name="top_plate">
+    <link name="${prefix}/top_plate">
       <inertial>
         <mass value="0.1"/>
@@ -63,14 +63,14 @@
       </visual>
     </link>
-    <gazebo reference="top_plate">
+    <gazebo reference="${prefix}/top_plate">
       <material>Gazebo/Black</material>
     </gazebo>
-    <joint name="base_top_joint" type="fixed">
+    <joint name="${prefix}/base_top_joint" type="fixed">
       <origin rpy="0 0 0" xyz="0.003 0 0.274"/>
-      <parent link="base_link"/>
-      <child link="top_plate"/>
+      <parent link="${prefix}/base_link"/>
+      <child link="${prefix}/top_plate"/>
     </joint>
     <!-- Front + Back Sonar -->
-    <link name="front_sonar">
+    <link name="${prefix}/front_sonar">
       <inertial>
         <mass value="0.1"/>
@@ -88,13 +88,13 @@
       </visual>
     </link>
-    <gazebo reference="front_sonar">
-      <material value="Gazebo/Yellow"/>
-    </gazebo>
-    <joint name="base_front_joint" type="fixed">
+    <gazebo reference="${prefix}/front_sonar">
+      <material value="Gazebo/Yellow"/>
+    </gazebo>
+    <joint name="${prefix}/base_front_joint" type="fixed">
       <origin rpy="0 0 0" xyz="0.193 0 0.25"/>
-      <parent link="base_link"/>
-      <child link="front_sonar"/>
-    </joint>
-    <link name="back_sonar">
+      <parent link="${prefix}/base_link"/>
+      <child link="${prefix}/front_sonar"/>
+    </joint>
+    <link name="${prefix}/back_sonar">
       <inertial>
         <mass value="0.1"/>
@@ -112,14 +112,14 @@
       </visual>
     </link>
-    <gazebo reference="back_sonar">
-      <material value="Gazebo/Yellow"/>
-    </gazebo>
-    <joint name="base_back_joint" type="fixed">
+    <gazebo reference="${prefix}/back_sonar">
+      <material value="Gazebo/Yellow"/>
+    </gazebo>
+    <joint name="${prefix}/base_back_joint" type="fixed">
       <origin rpy="0 0 0" xyz="-0.187 0 0.247"/>
-      <parent link="base_link"/>
-      <child link="back_sonar"/>
+      <parent link="${prefix}/base_link"/>
+      <child link="${prefix}/back_sonar"/>
     </joint>
     <!-- Front Axles + Wheels + Hubcaps -->
-    <link name="p3at_front_left_axle">
+    <link name="${prefix}/p3at_front_left_axle">
       <inertial>
         <mass value="0.1"/>
@@ -137,13 +137,13 @@
       </visual>
     </link>
-    <gazebo reference="p3at_front_left_axle">
+    <gazebo reference="${prefix}/p3at_front_left_axle">
       <material value="Gazebo/Grey"/>
     </gazebo>
-    <joint name="base_front_left_axle_joint" type="fixed">
+    <joint name="${prefix}/base_front_left_axle_joint" type="fixed">
       <origin rpy="0 0 0" xyz="0.135 0.156 0.111"/>
-      <parent link="base_link"/>
-      <child link="p3at_front_left_axle"/>
-    </joint>
-    <link name="p3at_front_left_hub">
+      <parent link="${prefix}/base_link"/>
+      <child link="${prefix}/p3at_front_left_axle"/>
+    </joint>
+    <link name="${prefix}/p3at_front_left_hub">
       <inertial>
         <mass value="0.1"/>
@@ -161,13 +161,13 @@
       </visual>
     </link>
-    <gazebo reference="p3at_front_left_hub">
-      <material value="Gazebo/Yellow"/>
-    </gazebo>
-    <joint name="base_front_left_hub_joint" type="fixed">
+    <gazebo reference="${prefix}/p3at_front_left_hub">
+      <material value="Gazebo/Yellow"/>
+    </gazebo>
+    <joint name="${prefix}/base_front_left_hub_joint" type="fixed">
       <origin rpy="0 0 0" xyz="0 0.041 0"/>
-      <parent link="p3at_front_left_axle"/>
-      <child link="p3at_front_left_hub"/>
-    </joint>
-    <link name="p3at_front_left_wheel">
+      <parent link="${prefix}/p3at_front_left_axle"/>
+      <child link="${prefix}/p3at_front_left_hub"/>
+    </joint>
+    <link name="${prefix}/p3at_front_left_wheel">
       <inertial>
         <mass value="1.2"/>
@@ -193,8 +193,8 @@
       </collision>
     </link>
-    <gazebo reference="p3at_front_left_wheel">
+    <gazebo reference="${prefix}/p3at_front_left_wheel">
       <material value="Gazebo/Black"/>
     </gazebo>
-    <joint name="p3at_front_left_wheel_joint" type="continuous">
+    <joint name="${prefix}/p3at_front_left_wheel_joint" type="continuous">
       <axis xyz="0 1 0"/>
       <anchor xyz="0 0 0"/>
@@ -202,9 +202,9 @@
       <joint_properties damping="0.7"/>
       <origin rpy="0 0 0" xyz="0 0 0"/>
-      <parent link="p3at_front_left_hub"/>
-      <child link="p3at_front_left_wheel"/>
+      <parent link="${prefix}/p3at_front_left_hub"/>
+      <child link="${prefix}/p3at_front_left_wheel"/>
     </joint>
     <!-- Back Axles + Wheels + Hubcaps -->
-    <link name="p3at_back_left_axle">
+    <link name="${prefix}/p3at_back_left_axle">
       <inertial>
         <mass value="0.1"/>
@@ -228,13 +228,13 @@
       </collision>
     </link>
-    <gazebo reference="p3at_back_left_axle">
+    <gazebo reference="${prefix}/p3at_back_left_axle">
       <material value="Gazebo/Grey"/>
     </gazebo>
-    <joint name="p3at_back_left_axle_joint" type="fixed">
+    <joint name="${prefix}/p3at_back_left_axle_joint" type="fixed">
       <origin rpy="0 0 0" xyz="-0.134 0.156 0.111"/>
-      <parent link="base_link"/>
-      <child link="p3at_back_left_axle"/>
-    </joint>
-    <link name="p3at_back_left_hub">
+      <parent link="${prefix}/base_link"/>
+      <child link="${prefix}/p3at_back_left_axle"/>
+    </joint>
+    <link name="${prefix}/p3at_back_left_hub">
       <inertial>
         <mass value="0.1"/>
@@ -256,13 +256,13 @@
       </collision>
     </link>
-    <gazebo reference="p3at_back_left_hub">
-      <material value="Gazebo/Yellow"/>
-    </gazebo>
-    <joint name="p3at_back_left_hub_joint" type="fixed">
+    <gazebo reference="${prefix}/p3at_back_left_hub">
+      <material value="Gazebo/Yellow"/>
+    </gazebo>
+    <joint name="${prefix}/p3at_back_left_hub_joint" type="fixed">
       <origin rpy="0 0 0" xyz="-0 0.041 0"/>
-      <parent link="p3at_back_left_axle"/>
-      <child link="p3at_back_left_hub"/>
-    </joint>
-    <link name="p3at_back_left_wheel">
+      <parent link="${prefix}/p3at_back_left_axle"/>
+      <child link="${prefix}/p3at_back_left_hub"/>
+    </joint>
+    <link name="${prefix}/p3at_back_left_wheel">
       <inertial>
         <mass value="1.2"/>
@@ -285,8 +285,8 @@
       </collision>
     </link>
-    <gazebo reference="p3at_back_left_wheel">
+    <gazebo reference="${prefix}/p3at_back_left_wheel">
       <material value="Gazebo/Black"/>
     </gazebo>
-    <joint name="p3at_back_left_wheel_joint" type="continuous">
+    <joint name="${prefix}/p3at_back_left_wheel_joint" type="continuous">
       <axis xyz="0 1 0"/>
       <anchor xyz="0 0 0"/>
@@ -294,9 +294,9 @@
       <joint_properties damping="0.7"/>
       <origin rpy="0 0 0" xyz="0 0 0"/>
-      <parent link="p3at_back_left_hub"/>
-      <child link="p3at_back_left_wheel"/>
+      <parent link="${prefix}/p3at_back_left_hub"/>
+      <child link="${prefix}/p3at_back_left_wheel"/>
     </joint>
     <!-- Front Axles + Wheels + Hubcaps -->
-    <link name="p3at_front_right_axle">
+    <link name="${prefix}/p3at_front_right_axle">
       <inertial>
         <mass value="0.1"/>
@@ -314,13 +314,13 @@
       </visual>
     </link>
-    <gazebo reference="p3at_front_right_axle">
+    <gazebo reference="${prefix}/p3at_front_right_axle">
       <material value="Gazebo/Grey"/>
     </gazebo>
-    <joint name="base_front_right_axle_joint" type="fixed">
+    <joint name="${prefix}/base_front_right_axle_joint" type="fixed">
       <origin rpy="0 0 0" xyz="0.135 -0.156 0.111"/>
-      <parent link="base_link"/>
-      <child link="p3at_front_right_axle"/>
-    </joint>
-    <link name="p3at_front_right_hub">
+      <parent link="${prefix}/base_link"/>
+      <child link="${prefix}/p3at_front_right_axle"/>
+    </joint>
+    <link name="${prefix}/p3at_front_right_hub">
       <inertial>
         <mass value="0.1"/>
@@ -338,13 +338,13 @@
       </visual>
     </link>
-    <gazebo reference="p3at_front_right_hub">
-      <material value="Gazebo/Yellow"/>
-    </gazebo>
-    <joint name="base_front_right_hub_joint" type="fixed">
+    <gazebo reference="${prefix}/p3at_front_right_hub">
+      <material value="Gazebo/Yellow"/>
+    </gazebo>
+    <joint name="${prefix}/base_front_right_hub_joint" type="fixed">
       <origin rpy="0 0 0" xyz="0 -0.041 0"/>
-      <parent link="p3at_front_right_axle"/>
-      <child link="p3at_front_right_hub"/>
-    </joint>
-    <link name="p3at_front_right_wheel">
+      <parent link="${prefix}/p3at_front_right_axle"/>
+      <child link="${prefix}/p3at_front_right_hub"/>
+    </joint>
+    <link name="${prefix}/p3at_front_right_wheel">
       <inertial>
         <mass value="1.2"/>
@@ -370,8 +370,8 @@
       </collision>
     </link>
-    <gazebo reference="p3at_front_right_wheel">
+    <gazebo reference="${prefix}/p3at_front_right_wheel">
       <material value="Gazebo/Black"/>
     </gazebo>
-    <joint name="p3at_front_right_wheel_joint" type="continuous">
+    <joint name="${prefix}/p3at_front_right_wheel_joint" type="continuous">
       <axis xyz="0 1 0"/>
       <anchor xyz="0 0 0"/>
@@ -379,9 +379,9 @@
       <joint_properties damping="0.7"/>
       <origin rpy="0 0 0" xyz="0 0 0"/>
-      <parent link="p3at_front_right_hub"/>
-      <child link="p3at_front_right_wheel"/>
+      <parent link="${prefix}/p3at_front_right_hub"/>
+      <child link="${prefix}/p3at_front_right_wheel"/>
     </joint>
     <!-- Back Axles + Wheels + Hubcaps -->
-    <link name="p3at_back_right_axle">
+    <link name="${prefix}/p3at_back_right_axle">
       <inertial>
         <mass value="0.1"/>
@@ -405,13 +405,13 @@
       </collision>
     </link>
-    <gazebo reference="p3at_back_right_axle">
+    <gazebo reference="${prefix}/p3at_back_right_axle">
       <material value="Gazebo/Grey"/>
     </gazebo>
-    <joint name="p3at_back_right_axle_joint" type="fixed">
+    <joint name="${prefix}/p3at_back_right_axle_joint" type="fixed">
       <origin rpy="0 0 0" xyz="-0.134 -0.156 0.111"/>
-      <parent link="base_link"/>
-      <child link="p3at_back_right_axle"/>
-    </joint>
-    <link name="p3at_back_right_hub">
+      <parent link="${prefix}/base_link"/>
+      <child link="${prefix}/p3at_back_right_axle"/>
+    </joint>
+    <link name="${prefix}/p3at_back_right_hub">
       <inertial>
         <mass value="0.1"/>
@@ -433,13 +433,13 @@
       </collision>
     </link>
-    <gazebo reference="p3at_back_right_hub">
-      <material value="Gazebo/Yellow"/>
-    </gazebo>
-    <joint name="p3at_back_right_hub_joint" type="fixed">
+    <gazebo reference="${prefix}/p3at_back_right_hub">
+      <material value="Gazebo/Yellow"/>
+    </gazebo>
+    <joint name="${prefix}/p3at_back_right_hub_joint" type="fixed">
       <origin rpy="0 0 0" xyz="-0 -0.041 0"/>
-      <parent link="p3at_back_right_axle"/>
-      <child link="p3at_back_right_hub"/>
-    </joint>
-    <link name="p3at_back_right_wheel">
+      <parent link="${prefix}/p3at_back_right_axle"/>
+      <child link="${prefix}/p3at_back_right_hub"/>
+    </joint>
+    <link name="${prefix}/p3at_back_right_wheel">
       <inertial>
         <mass value="1.2"/>
@@ -462,8 +462,8 @@
       </collision>
     </link>
-    <gazebo reference="p3at_back_right_wheel">
+    <gazebo reference="${prefix}/p3at_back_right_wheel">
       <material value="Gazebo/Black"/>
     </gazebo>
-    <joint name="p3at_back_right_wheel_joint" type="continuous">
+    <joint name="${prefix}/p3at_back_right_wheel_joint" type="continuous">
       <axis xyz="0 1 0"/>
       <anchor xyz="0 0 0"/>
@@ -471,8 +471,14 @@
       <joint_properties damping="0.7"/>
       <origin rpy="0 0 0" xyz="0 0 0"/>
-      <parent link="p3at_back_right_hub"/>
-      <child link="p3at_back_right_wheel"/>
-    </joint>
-  <!-- Gazebo -->
+      <parent link="${prefix}/p3at_back_right_hub"/>
+      <child link="${prefix}/p3at_back_right_wheel"/>
+    </joint>
+    <!-- Gazebo -->
+    <xacro:include filename="$(find follower_description)/urdf/gazebo.urdf.xacro" />
+    <xacro:p3at_control prefix="${prefix}" />
+    <xacro:p3at_wheel link="${prefix}/p3at_front_left_wheel_link" />
+    <xacro:p3at_wheel link="${prefix}/p3at_front_right_wheel_link" />
+    <xacro:p3at_wheel link="${prefix}/p3at_back_left_wheel_link" />
+    <xacro:p3at_wheel link="${prefix}/p3at_back_right_wheel_link" />
   </xacro:macro>
 </robot>

Commit message: MG: working laser

File: follower_description/urdf/gazebo.urdf.xacro (robot description, xacro)
@@ -21,7 +21,4 @@
             </plugin>
         </gazebo>
-      <!-- <gazebo>
-        <plugin name="joint_state_publisher" filename="libgazebo_ros_joint_state_publisher.so" />
-      </gazebo> -->
     </xacro:macro>
     <xacro:macro name='p3at_wheel' params='link'>
@@ -176,3 +173,36 @@
     </gazebo>
   </xacro:macro>
+	<xacro:macro name="sensor_hokuyo_urg_gazebo" params="name">
+		<gazebo reference="${name}_link">
+			<sensor type="gpu_ray" name="${name}_sensor">
+				<pose>0 0 0 0 0 0</pose>
+				<visualize>true</visualize>
+				<update_rate>10</update_rate>
+				<ray>
+					<scan>
+						<horizontal>
+							<samples>640</samples>
+							<resolution>1</resolution>
+							<min_angle>-2.0943</min_angle>
+							<max_angle>2.0943</max_angle>
+						</horizontal>
+					</scan>
+					<range>
+						<min>0.02</min>
+						<max>4.0</max>
+						<resolution>0.00628318531</resolution>
+					</range>
+					<noise>
+						<type>gaussian</type>
+						<mean>0.0</mean>
+						<stddev>0.01</stddev>
+					</noise>
+				</ray>
+				<plugin name="${name}_controller" filename="libgazebo_ros_gpu_laser.so">
+					<topicName>${name}/scan</topicName>
+					<frameName>${name}_link</frameName>
+				</plugin>
+			</sensor>
+		</gazebo>
+	</xacro:macro>
 </robot>
